File: eagle/feedback-strobe.brd (EAGLE design)
At the start: 39.9 x 27.9 mm, 21 parts, among them J2 MOTOR, U1 STN3NF06L, U2 +12v

Commit message: added new voltage regulator, reduced number of vias, added more spacing between traces.
Parts:
- removed U2: +12v, SparkFun-PowerIC:TO-252
- added U$1: V_REG_MIC2920, SparkFun-PowerIC:SOT223
- R9: value (none) -> 10k
- moved R9 12.0 mm to (7.98, 5.69), flipped to the bottom, turned to 180 degrees
- moved U1 9.46 mm to (13.3, 12.5)
- moved C1 5.95 mm to (16.5, 20.6), turned to 0 degrees
- moved J2 1.02 mm to (23.6, 24.1)
Connections:
- removed net N$8: J2.2
- new net N$7: J2.2, U1.2
- net 5V: no longer U2.2
- net GND: now also U$1.2, U1.3; no longer U2.3
- net VCC: now also U$1.3
- net VIN: now also U$1.1; no longer U2.1
Routing:
- net N$7: track 0.00 -> 16.5 mm
- net N$4: track 13.9 -> 0.00 mm, vias 1 -> 0
- net VIN: track 43.4 -> 32.8 mm
- net VCC: track 0.00 -> 8.75 mm, vias 0 -> 1
- net GND: track 36.4 -> 30.4 mm, vias 4 -> 2
- net MOTOR_CTRL: track 3.31 -> 9.06 mm, vias 0 -> 1
- net N$8: track 3.07 -> 0.00 mm
- net LED1: track 16.2 -> 17.2 mm
- net 5V: track 11.4 -> 10.6 mm

Commit message: put my name on the board
Parts:
- turned U1 to 45 degrees
Routing:
- net N$7: track 16.5 -> 15.7 mm
- net MOTOR_CTRL: track 9.06 -> 9.64 mm
Other:
- board text added: "Ruffner"
Changed lines of the file:
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@@
 <dimension x1="0" y1="0" x2="39.878" y2="0" x3="19.939" y3="-3.81" textsize="1.778" layer="1"/>
 <dimension x1="0" y1="0" x2="0" y2="27.94" x3="-7.62" y3="13.97" textsize="1.778" layer="1"/>
+<text x="38.608" y="24.13" size="2.54" layer="16" rot="MR0">Ruffner</text>
 </plain>
 <attributes>
@@
 <element name="J1" library="SparkFun-Connectors" package="1X03" value="" x="3.048" y="6.223" rot="R90"/>
 <element name="U$1" library="SparkFun-PowerIC" package="SOT223" value="V_REG_MIC2920" x="31.5976" y="9.144" rot="R270"/>
-<element name="U1" library="n-fet" package="SOT-223" value="STN3NF06L" x="13.335" y="12.4968">
-<attribute name="RDSONMAXIDVGS" value="100 mOhm  1.5A 10V" x="13.335" y="12.4968" size="1.778" layer="27" display="off"/>
-<attribute name="DATASHEET" value="httpwww.st.cominternetcomTECHNICAL_RESOURCESTECHNICAL_LITERATUREDATASHEETCD00002430.pdf" x="13.335" y="12.4968" size="1.778" layer="27" display="off"/>
-<attribute name="VGSTHMAXID" value="2.8V  250µA" x="13.335" y="12.4968" size="1.778" layer="27" display="off"/>
-<attribute name="MANUFACTURER_PART_NUMBER" value="STN3NF06L" x="13.335" y="12.4968" size="1.778" layer="27" display="off"/>
-<attribute name="CATEGORY" value="" x="13.335" y="12.4968" size="1.778" layer="27" display="off"/>
-<attribute name="DRAINTOSOURCEVOLTAGEVDSS" value="60V" x="13.335" y="12.4968" size="1.778" layer="27" display="off"/>
-<attribute name="QUANTITY_AVAILABLE" value="16000" x="13.335" y="12.4968" size="1.778" layer="27" display="off"/>
-<attribute name="FETTYPE" value="MOSFET NChannel Metal Oxide" x="13.335" y="12.4968" size="1.778" layer="27" display="off"/>
-<attribute name="SUPPLIERDEVICEPACKAGE" value="SOT223" x="13.335" y="12.4968" size="1.778" layer="27" display="off"/>
-<attribute name="PACKAGECASE" value="TO2614 TO261AA" x="13.335" y="12.4968" size="1.778" layer="27" display="off"/>
-<attribute name="PACKAGING" value="Tape &amp;amp Reel TR" x="13.335" y="12.4968" size="1.778" layer="27" display="off"/>
-<attribute name="VENDOR" value="ST Microelectronics" x="13.335" y="12.4968" size="1.778" layer="27" display="off"/>
-<attribute name="CURRENTCONTINUOUSDRAINID25C" value="4A" x="13.335" y="12.4968" size="1.778" layer="27" display="off"/>
-<attribute name="MOUNTINGTYPE" value="Surface Mount" x="13.335" y="12.4968" size="1.778" layer="27" display="off"/>
-<attribute name="POWERMAX" value="3.3W" x="13.335" y="12.4968" size="1.778" layer="27" display="off"/>
-<attribute name="COPYRIGHT" value="Copyright C 2015 Accelerated Designs. All rights reserved" x="13.335" y="12.4968" size="1.778" layer="27" display="off"/>
-<attribute name="DIGIKEYPARTNUMBER" value="49731772ND" x="13.335" y="12.4968" size="1.778" layer="27" display="off"/>
-<attribute name="GATECHARGEQGVGS" value="9nC  5V" x="13.335" y="12.4968" size="1.778" layer="27" display="off"/>
-<attribute name="FETFEATURE" value="Logic Level Gate" x="13.335" y="12.4968" size="1.778" layer="27" display="off"/>
-<attribute name="INPUTCAPACITANCECISSVDS" value="340pF  25V" x="13.335" y="12.4968" size="1.778" layer="27" display="off"/>
+<element name="U1" library="n-fet" package="SOT-223" value="STN3NF06L" x="13.335" y="12.4968" rot="R45">
+<attribute name="RDSONMAXIDVGS" value="100 mOhm  1.5A 10V" x="13.335" y="12.4968" size="1.778" layer="27" rot="R45" display="off"/>
+<attribute name="DATASHEET" value="httpwww.st.cominternetcomTECHNICAL_RESOURCESTECHNICAL_LITERATUREDATASHEETCD00002430.pdf" x="13.335" y="12.4968" size="1.778" layer="27" rot="R45" display="off"/>
+<attribute name="VGSTHMAXID" value="2.8V  250µA" x="13.335" y="12.4968" size="1.778" layer="27" rot="R45" display="off"/>
+<attribute name="MANUFACTURER_PART_NUMBER" value="STN3NF06L" x="13.335" y="12.4968" size="1.778" layer="27" rot="R45" display="off"/>
+<attribute name="CATEGORY" value="" x="13.335" y="12.4968" size="1.778" layer="27" rot="R45" display="off"/>
+<attribute name="DRAINTOSOURCEVOLTAGEVDSS" value="60V" x="13.335" y="12.4968" size="1.778" layer="27" rot="R45" display="off"/>
+<attribute name="QUANTITY_AVAILABLE" value="16000" x="13.335" y="12.4968" size="1.778" layer="27" rot="R45" display="off"/>
+<attribute name="FETTYPE" value="MOSFET NChannel Metal Oxide" x="13.335" y="12.4968" size="1.778" layer="27" rot="R45" display="off"/>
+<attribute name="SUPPLIERDEVICEPACKAGE" value="SOT223" x="13.335" y="12.4968" size="1.778" layer="27" rot="R45" display="off"/>
+<attribute name="PACKAGECASE" value="TO2614 TO261AA" x="13.335" y="12.4968" size="1.778" layer="27" rot="R45" display="off"/>
+<attribute name="PACKAGING" value="Tape &amp;amp Reel TR" x="13.335" y="12.4968" size="1.778" layer="27" rot="R45" display="off"/>
+<attribute name="VENDOR" value="ST Microelectronics" x="13.335" y="12.4968" size="1.778" layer="27" rot="R45" display="off"/>
+<attribute name="CURRENTCONTINUOUSDRAINID25C" value="4A" x="13.335" y="12.4968" size="1.778" layer="27" rot="R45" display="off"/>
+<attribute name="MOUNTINGTYPE" value="Surface Mount" x="13.335" y="12.4968" size="1.778" layer="27" rot="R45" display="off"/>
+<attribute name="POWERMAX" value="3.3W" x="13.335" y="12.4968" size="1.778" layer="27" rot="R45" display="off"/>
+<attribute name="COPYRIGHT" value="Copyright C 2015 Accelerated Designs. All rights reserved" x="13.335" y="12.4968" size="1.778" layer="27" rot="R45" display="off"/>
+<attribute name="DIGIKEYPARTNUMBER" value="49731772ND" x="13.335" y="12.4968" size="1.778" layer="27" rot="R45" display="off"/>
+<attribute name="GATECHARGEQGVGS" value="9nC  5V" x="13.335" y="12.4968" size="1.778" layer="27" rot="R45" display="off"/>
+<attribute name="FETFEATURE" value="Logic Level Gate" x="13.335" y="12.4968" size="1.778" layer="27" rot="R45" display="off"/>
+<attribute name="INPUTCAPACITANCECISSVDS" value="340pF  25V" x="13.335" y="12.4968" size="1.778" layer="27" rot="R45" display="off"/>
 </element>
 <element name="R9" library="SparkFun-Passives" package="0603-RES" value="10k" x="7.9756" y="5.6896" rot="MR180"/>
@@
 <contactref element="J1" pad="3"/>
 <via x="20.066" y="5.842" extent="1-16" drill="0.6" shape="square"/>
-<wire x1="33.909" y1="2.794" x2="35.433" y2="1.27" width="0.6096" layer="1"/>
-<wire x1="35.433" y1="1.27" x2="38.608" y2="1.27" width="0.6096" layer="1"/>
-<wire x1="38.608" y1="1.27" x2="38.608" y2="8.382" width="0.6096" layer="1"/>
-<wire x1="38.608" y1="8.382" x2="37.592" y2="9.398" width="0.6096" layer="1"/>
-<wire x1="37.846" y1="11.978" x2="37.846" y2="25.654" width="0.6096" layer="1"/>
-<wire x1="37.846" y1="25.654" x2="37.734" y2="25.766" width="0.6096" layer="1"/>
-<wire x1="37.734" y1="25.766" x2="35.052" y2="25.766" width="0.6096" layer="1"/>
 <via x="9.652" y="7.62" extent="1-16" drill="0.6" shape="square"/>
 <contactref element="U$1" pad="2"/>
 <contactref element="U1" pad="3"/>
 <contactref element="R9" pad="1"/>
+<wire x1="33.909" y1="2.794" x2="33.782" y2="2.667" width="0.4064" layer="1"/>
+<wire x1="33.782" y1="2.667" x2="33.782" y2="1.27" width="0.4064" layer="1"/>
+<wire x1="33.782" y1="1.27" x2="38.608" y2="1.27" width="0.4064" layer="1"/>
+<wire x1="38.608" y1="1.27" x2="38.354" y2="1.524" width="0.4064" layer="1"/>
+<wire x1="38.354" y1="1.524" x2="38.354" y2="11.938" width="0.4064" layer="1"/>
+<wire x1="38.354" y1="11.938" x2="31.496" y2="11.938" width="0.4064" layer="1"/>
+<wire x1="31.496" y1="11.938" x2="31.75" y2="11.684" width="0.4064" layer="1"/>
+<wire x1="31.75" y1="11.684" x2="31.75" y2="9.144" width="0.4064" layer="1"/>
+<wire x1="31.75" y1="9.144" x2="28.4988" y2="9.144" width="0.4064" layer="1"/>
 </signal>
 <signal name="VIN">
@@
 <wire x1="11.176" y1="5.842" x2="11.176" y2="2.794" width="0.254" layer="16"/>
 <wire x1="11.176" y1="5.842" x2="11.035" y2="5.842" width="0.3048" layer="1"/>
-<wire x1="11.035" y1="5.842" x2="11.035" y2="9.2964" width="0.3048" layer="1"/>
+<wire x1="11.035" y1="5.842" x2="13.971678125" y2="8.607428125" width="0.3048" layer="1"/>
 </signal>
 <signal name="N$8">
@@
 <contactref element="J2" pad="2"/>
 <contactref element="U1" pad="2"/>
-<wire x1="23.622" y1="21.59" x2="20.32" y2="18.288" width="0.6096" layer="1"/>
-<wire x1="20.32" y1="18.288" x2="18.288" y2="16.002" width="0.6096" layer="1"/>
-<wire x1="18.288" y1="16.002" x2="13.335" y2="11.049" width="0.6096" layer="1"/>
-<wire x1="13.335" y1="11.049" x2="13.335" y2="9.2964" width="0.6096" layer="1"/>
+<wire x1="23.622" y1="21.59" x2="14.478" y2="12.446" width="0.6096" layer="1"/>
+<wire x1="14.478" y1="12.446" x2="14.478" y2="11.176" width="0.6096" layer="1"/>
+<wire x1="14.478" y1="11.176" x2="15.420225" y2="10.233775" width="0.6096" layer="1"/>
+<wire x1="15.420225" y1="10.233775" x2="15.598021875" y2="10.233775" width="0.6096" layer="1"/>
 </signal>
 </signals>
